File: docs/hardware/schematic/msp430_gameboy.kicad_sch (KiCad schematic)
At the start: 32 parts, among them J1 SSD1325_OLED, J2 LiPo_Charger, SW1 BTN_A, SW2 BTN_B, SW3 BTN_C, SW4 BTN_D, SW5 BTN_E, SW6 BTN_F, SW7 BTN_G, SW8 BTN_H, U1 MSP430G2553, U2 SN74HC165N, U3 LM386N-1, U4 23LC1024-I/P, U5 W25Q128JVSSIQ

Commit message: fix: resolve 'extends' into standalone symbols for schematic lib_symbols
KiCad does not support 'extends' inside a schematic's lib_symbols section —
it only works in .kicad_sym library files. The new extract_sym() resolver:
- Detects (extends "PARENT") in the child symbol block
- Extracts the parent's body/pin sub-symbols and the child's properties
- Renames parent sub-symbols to use the child's name (NAME_0_1 → ChildName_0_1)
- Assembles a fully standalone symbol with no 'extends' dependency
- Also strips 'embedded_fonts' which is likewise invalid in lib_symbols

Co-Authored-By: Claude Sonnet 4.6 <noreply@anthropic.com>
Connections:
- net BTN_A: now also U2.11 (D0)
- net BTN_B: now also U2.12 (D1)
- net BTN_C: now also U2.13 (D2)
- net BTN_D: now also U2.14 (D3)
- net BTN_E: now also U2.3 (D4)
- net BTN_F: now also U2.4 (D5)
- net BTN_G: now also U2.5 (D6)
- net BTN_H: now also U2.6 (D7)
- net FLASH_CS: now also U1.12 (P2.4/TA1.2), U5.1 (~{CS})
- net GND: now also U1.20 (DVSS), U2.10 (DS), U2.15 (~{CE}), U2.8 (GND), U5.4 (GND)
- net MISO: now also U1.14 (TDI/TCLK/UCB0SOMI/UCB0SCL/TA0.1/CA6/A6/P1.6), U2.9 (Q7), U5.2 (DO/IO_{1})
- net MOSI: now also U1.15 (TDO/TDI/UCB0SIMO/UCB0SDA/CAOUT/CA7/A7/P1.7), U5.5 (DI/IO_{0})
- net OLED_CS: now also U1.8 (P2.0/TA1.0)
- net OLED_DC: now also U1.9 (P2.1/TA1.1)
- net OLED_RST: now also U1.10 (P2.2/TA1.1)
- net PWM_OUT: now also U1.4 (UCA0TXD/UCA0SIMO/TA0.1/CA2/A2/P1.2)
- net SCK: now also U1.7 (TMS/UCB0CLK/UCA0STE/TA0.0/CA5/A5/P1.5), U2.2 (CP), U5.6 (CLK)
- net SH_LD: now also U1.13 (P2.5/TA1.2), U2.1 (~{PL})
- net SRAM_CS: now also U1.11 (P2.3/TA1.0)
- net VCC: now also U1.1 (DVCC), U2.16 (VCC), U5.3 (~{WP}/IO_{2}), U5.7 (~{HOLD}/~{RESET}/IO_{3}), U5.8 (VCC)
