File: docs/hardware/schematic/msp430_gameboy.kicad_sch (KiCad schematic)
At the start: 32 parts, among them J1 SSD1325_OLED, J2 LiPo_Charger, SW1 BTN_A, SW2 BTN_B, SW3 BTN_C, SW4 BTN_D, SW5 BTN_E, SW6 BTN_F, SW7 BTN_G, SW8 BTN_H, U1 MSP430G2553, U2 SN74HC165N, U3 LM386N-1, U4 23LC1024-I/P, U5 W25Q128JVSSIQ

Commit message: course: remove solution dirs, reduce exercise scaffolding; update schematic
Exercise format changes:
- Delete all solution/ directories (lessons 01, 02, 04)
- Lesson 04 ex2: remove GCD walkthrough and pseudocode structure hint
- Lesson 04 ex3: remove all templates and pre-computed constants; spec only
- Lesson 04 README: note cumulative knowledge requirements per exercise
- Student completed ex1 (10/10) and ex2 (10/10); ex3 in progress

Schematic (gen_kicad7.py / msp430_gameboy.kicad_sch):
- Replace SSD1306 module with full OLED-128O064D discrete circuit
- Add TP4056 + DW01A + back-to-back NMOS LiPo charger/protection circuit
- Add 20 explicit junction elements for T-intersections
- CE and TEMP tied to VBUS (5V) not VCC (3.3V)

Co-Authored-By: Claude Sonnet 4.6 <noreply@anthropic.com>
Parts:
- removed J1: SSD1325_OLED, symbol Conn_OLED_7
- removed J2: LiPo_Charger, symbol Conn_LiPo_4
- removed LS1: SP-3605, symbol Speaker
- removed SW1: BTN_A, symbol SW_Push
- removed SW2: BTN_B, symbol SW_Push
- removed SW3: BTN_C, symbol SW_Push
- removed SW4: BTN_D, symbol SW_Push
- removed SW5: BTN_E, symbol SW_Push
- removed SW6: BTN_F, symbol SW_Push
- removed SW7: BTN_G, symbol SW_Push
- removed SW8: BTN_H, symbol SW_Push
- added BT1: LiPo_JST, symbol Connector:Conn_01x02_Pin
- added C10, C11: 4.7uF 10V X5R, symbol Device:C
- added C12: 100nF 16V X7R, symbol Device:C
- added C13: 10uF 16V X5R, symbol Device:C
- added C14: 10uF 10V X5R, symbol Device:C
- added C15, C16, C9: 1uF 10V X5R, symbol Device:C
- added C8: 100nF 10V X5R, symbol Device:C
- added D1: LED_RED 0603, symbol Device:LED
- added D2: LED_GRN 0603, symbol Device:LED
- added DS1: OLED-128O064D, symbol Display_Graphic:OLED-128O064D
- added J4: USB_B_Micro, symbol Connector:USB_B_Micro
- added LS1: SP-3605, symbol Device:Speaker
- added Q1, Q2: AO3400, symbol Transistor_FET:Q_NMOS_GSD
- added R10: 910k 1% 0402, symbol Device:R
- added R11: 2k 1%, symbol Device:R
- added R12, R13: 1k 5%, symbol Device:R
- added SW1: BTN_A, symbol Switch:SW_Push
- added SW2: BTN_B, symbol Switch:SW_Push
- added SW3: BTN_C, symbol Switch:SW_Push
- added SW4: BTN_D, symbol Switch:SW_Push
- added SW5: BTN_E, symbol Switch:SW_Push
- added SW6: BTN_F, symbol Switch:SW_Push
- added SW7: BTN_G, symbol Switch:SW_Push
- added SW8: BTN_H, symbol Switch:SW_Push
- added U7: TP4056-42-ESOP8, symbol Battery_Management:TP4056-42-ESOP8
- added U8: DW01A, symbol Battery_Management:DW01A
Connections:
- net GND: now also C10.2, C11.1, C12.2, C13.2, C14.2, DS1.1 (GND), DS1.10 (BS0), DS1.11 (BS1), DS1.29 (VLSS), DS1.30 (GND), DS1.8 (VSS), J4.5 (GND), J4.6 (Shield), LS1.2, Q2.2 (S), R11.2, SW1.1, SW2.1, SW3.1, SW4.1, SW5.1, SW6.1, SW7.1, SW8.1, U7.3 (GND), U7.9 (EPAD), U8.2 (CS), U8.6 (GND)
- net MOSI: now also DS1.19 (D1)
- net OLED_CS: now also DS1.13 (~{CS})
- net OLED_DC: now also DS1.15 (D/~{C})
- net OLED_RST: now also DS1.14 (~{RES})
- net SCK: now also DS1.18 (D0)
- net VCC: now also C8.1, C9.1, DS1.12 (BS2), R10.1, R12.1, R13.1
- net BTN_A: no longer names the net of R2.2, U2.11 (D0)
- net BTN_A: now also SW1.2
- net BTN_B: no longer names the net of R3.2, U2.12 (D1)
- net BTN_B: now also SW2.2
- net BTN_C: no longer names the net of R4.2, U2.13 (D2)
- net BTN_C: now also SW3.2
- net BTN_D: no longer names the net of R5.2, U2.14 (D3)
- net BTN_D: now also SW4.2
- net BTN_E: no longer names the net of R6.2, U2.3 (D4)
- net BTN_E: now also SW5.2
- net BTN_F: no longer names the net of R7.2, U2.4 (D5)
- net BTN_F: now also SW6.2
- net BTN_G: no longer names the net of R8.2, U2.5 (D6)
- net BTN_G: now also SW7.2
- net BTN_H: no longer names the net of R9.2, U2.6 (D7)
- net BTN_H: now also SW8.2
- net FILT_MID: no longer names the net of C5.1, R1.2
- net LM386_BYP: no longer names the net of C6.2, U3.7 (BYPASS)
- net SPK_OUT: no longer names the net of C7.1
- net SPK_OUT: now also LS1.1; no longer U3.5
- net SPK_RAW: no longer names the net of C7.2
- net SPK_RAW: now also U3.5
- net VOL_WIPER: no longer names the net of C5.2, U3.3 (+)
- new net: C8.2, DS1.9 (VDD)
- new net: R11.1, U7.2 (PROG)
- new net: C11.2, DS1.27 (VCOMH)
- new net: D2.1 (K), U7.6 (~{STDBY})
- new net: D2.2 (A), R13.2
- new net: Q2.1 (G), U8.3 (OC)
- new net: Q1.3 (D), Q2.3 (D)
- new net: C9.2, DS1.6 (VBAT)
- new net: C16.1, DS1.5 (C1N)
- new net: C16.2, DS1.4 (C1P)
- new net: D1.1 (K), U7.7 (~{CHRG})
- new net: D1.2 (A), R12.2
- new net: BT1.2 (Pin_2), Q1.2 (S)
- new net: C15.1, DS1.2 (C2N)
- new net: C15.2, DS1.3 (C2P)
- new net: C10.1, DS1.28 (VCC)
- new net: DS1.26 (IREF), R10.2
- new net: Q1.1 (G), U8.1 (OD)
- new net VBAT: BT1.1 (Pin_1), C14.1, U7.5 (BAT), U8.5 (VCC)
- new net VBUS: C12.1, C13.1, J4.1 (VBUS), U7.1 (TEMP), U7.4 (V_{CC}), U7.8 (CE)
- no-connect marks 12 -> 24
